File: KiCad/nixie.sch (KiCad schematic (older format))
At the start: 17 parts, among them U2 TLP627-2, U3 SN74141, U4 TLP627-2, U5 TLP627-2

Commit message: change schematics
Parts:
- added D3, D4, D5, D6, D7, D8: LED, symbol LED
- added R14, R15, R16, R17, R18, R19: 300, Resistors_SMD:R_0603_HandSoldering, symbol R
- NT1, NT2, NT3, NT4, NT5, NT6: footprint (none) -> nixie_clock:IN-12
- R1, R3, R4, R5, R6, R7: footprint Resistors_ThroughHole:R_Axial_DIN0207_L6.3mm_D2.5mm_P10.16mm_Horizontal -> Resistors_SMD:R_0603_HandSoldering
Connections:
- net +3V3: now also R14.2, R15.2, R16.2, R17.2, R18.2, R19.2
- new net: D3.2 (A), R14.1
- new net: D4.2 (A), R15.1
- new net: D5.2 (A), R16.1
- new net: D6.2 (A), R17.1
- new net: D7.2 (A), R18.1
- new net: D8.2 (A), R19.1
- new net led0: D3.1 (K)
- new net led1: D4.1 (K)
- new net led2: D5.1 (K)
- new net led3: D6.1 (K)
- new net led4: D7.1 (K)
- new net led5: D8.1 (K)
Changed lines of the file:
@@
 F 0 "NT1" H 2300 4100 60  0000 C CNN
 F 1 "IN-12B" H 1500 4100 60  0000 C CNN
-F 2 "" H 1700 3700 60  0001 C CNN
+F 2 "nixie_clock:IN-12" H 1700 3700 60  0001 C CNN
 F 3 "" H 1700 3700 60  0000 C CNN
 	1    1700 3700
@@
 F 0 "NT2" H 3800 4100 60  0000 C CNN
 F 1 "IN-12B" H 3000 4100 60  0000 C CNN
-F 2 "" H 3200 3700 60  0001 C CNN
+F 2 "nixie_clock:IN-12" H 3200 3700 60  0001 C CNN
 F 3 "" H 3200 3700 60  0000 C CNN
 	1    3200 3700
@@
 F 0 "NT3" H 5300 4100 60  0000 C CNN
 F 1 "IN-12B" H 4500 4100 60  0000 C CNN
-F 2 "" H 4700 3700 60  0001 C CNN
+F 2 "nixie_clock:IN-12" H 4700 3700 60  0001 C CNN
 F 3 "" H 4700 3700 60  0000 C CNN
 	1    4700 3700
@@
 F 0 "NT4" H 6800 4100 60  0000 C CNN
 F 1 "IN-12B" H 6000 4100 60  0000 C CNN
-F 2 "" H 6200 3700 60  0001 C CNN
+F 2 "nixie_clock:IN-12" H 6200 3700 60  0001 C CNN
 F 3 "" H 6200 3700 60  0000 C CNN
 	1    6200 3700
@@
 F 0 "NT5" H 8300 4100 60  0000 C CNN
 F 1 "IN-12B" H 7500 4100 60  0000 C CNN
-F 2 "" H 7700 3700 60  0001 C CNN
+F 2 "nixie_clock:IN-12" H 7700 3700 60  0001 C CNN
 F 3 "" H 7700 3700 60  0000 C CNN
 	1    7700 3700
@@
 F 0 "NT6" H 9800 4100 60  0000 C CNN
 F 1 "IN-12B" H 9000 4100 60  0000 C CNN
-F 2 "" H 9200 3700 60  0001 C CNN
+F 2 "nixie_clock:IN-12" H 9200 3700 60  0001 C CNN
 F 3 "" H 9200 3700 60  0000 C CNN
 	1    9200 3700
@@
 F 0 "R1" V 980 2050 50  0000 C CNN
 F 1 "300" V 900 2050 50  0000 C CNN
-F 2 "Resistors_ThroughHole:R_Axial_DIN0207_L6.3mm_D2.5mm_P10.16mm_Horizontal" V 830 2050 50  0001 C CNN
+F 2 "Resistors_SMD:R_0603_HandSoldering" V 830 2050 50  0001 C CNN
 F 3 "" H 900 2050 50  0000 C CNN
 	1    900  2050
@@
 F 0 "R3" V 2530 2050 50  0000 C CNN
 F 1 "300" V 2450 2050 50  0000 C CNN
-F 2 "Resistors_ThroughHole:R_Axial_DIN0207_L6.3mm_D2.5mm_P10.16mm_Horizontal" V 2380 2050 50  0001 C CNN
+F 2 "Resistors_SMD:R_0603_HandSoldering" V 2380 2050 50  0001 C CNN
 F 3 "" H 2450 2050 50  0000 C CNN
 	1    2450 2050
@@
 F 0 "R4" V 4030 2050 50  0000 C CNN
 F 1 "300" V 3950 2050 50  0000 C CNN
-F 2 "Resistors_ThroughHole:R_Axial_DIN0207_L6.3mm_D2.5mm_P10.16mm_Horizontal" V 3880 2050 50  0001 C CNN
+F 2 "Resistors_SMD:R_0603_HandSoldering" V 3880 2050 50  0001 C CNN
 F 3 "" H 3950 2050 50  0000 C CNN
 	1    3950 2050
@@
 F 0 "R5" V 5530 2050 50  0000 C CNN
 F 1 "300" V 5450 2050 50  0000 C CNN
-F 2 "Resistors_ThroughHole:R_Axial_DIN0207_L6.3mm_D2.5mm_P10.16mm_Horizontal" V 5380 2050 50  0001 C CNN
+F 2 "Resistors_SMD:R_0603_HandSoldering" V 5380 2050 50  0001 C CNN
 F 3 "" H 5450 2050 50  0000 C CNN
 	1    5450 2050
@@
 F 0 "R6" V 7030 2050 50  0000 C CNN
 F 1 "300" V 6950 2050 50  0000 C CNN
-F 2 "Resistors_ThroughHole:R_Axial_DIN0207_L6.3mm_D2.5mm_P10.16mm_Horizontal" V 6880 2050 50  0001 C CNN
+F 2 "Resistors_SMD:R_0603_HandSoldering" V 6880 2050 50  0001 C CNN
 F 3 "" H 6950 2050 50  0000 C CNN
 	1    6950 2050
@@
 F 0 "R7" V 8530 2050 50  0000 C CNN
 F 1 "300" V 8450 2050 50  0000 C CNN
-F 2 "Resistors_ThroughHole:R_Axial_DIN0207_L6.3mm_D2.5mm_P10.16mm_Horizontal" V 8380 2050 50  0001 C CNN
+F 2 "Resistors_SMD:R_0603_HandSoldering" V 8380 2050 50  0001 C CNN
 F 3 "" H 8450 2050 50  0000 C CNN
 	1    8450 2050
@@
 NoConn ~ 8400 3800
 NoConn ~ 9900 3800
+$Comp
+L LED D3
+U 1 1 59EA2EC3
+P 5200 5750
+F 0 "D3" H 5200 5850 50  0000 C CNN
+F 1 "LED" H 5200 5650 50  0000 C CNN
+F 2 "" H 5200 5750 50  0000 C CNN
+F 3 "" H 5200 5750 50  0000 C CNN
+	1    5200 5750
+	1    0    0    -1
+$EndComp
+$Comp
+L LED D4
+U 1 1 59EA3159
+P 5200 6050
+F 0 "D4" H 5200 6150 50  0000 C CNN
+F 1 "LED" H 5200 5950 50  0000 C CNN
+F 2 "" H 5200 6050 50  0000 C CNN
+F 3 "" H 5200 6050 50  0000 C CNN
+	1    5200 6050
+	1    0    0    -1
+$EndComp
+$Comp
+L LED D5
+U 1 1 59EA3211
+P 5200 6350
+F 0 "D5" H 5200 6450 50  0000 C CNN
+F 1 "LED" H 5200 6250 50  0000 C CNN
+F 2 "" H 5200 6350 50  0000 C CNN
+F 3 "" H 5200 6350 50  0000 C CNN
+	1    5200 6350
+	1    0    0    -1
+$EndComp
+$Comp
+L LED D6
+U 1 1 59EA3217
+P 5200 6650
+F 0 "D6" H 5200 6750 50  0000 C CNN
+F 1 "LED" H 5200 6550 50  0000 C CNN
+F 2 "" H 5200 6650 50  0000 C CNN
+F 3 "" H 5200 6650 50  0000 C CNN
+	1    5200 6650
+	1    0    0    -1
+$EndComp
+$Comp
+L LED D7
+U 1 1 59EA33CB
+P 5200 6950
+F 0 "D7" H 5200 7050 50  0000 C CNN
+F 1 "LED" H 5200 6850 50  0000 C CNN
+F 2 "" H 5200 6950 50  0000 C CNN
+F 3 "" H 5200 6950 50  0000 C CNN
+	1    5200 6950
+	1    0    0    -1
+$EndComp
+$Comp
+L LED D8
+U 1 1 59EA33D1
+P 5200 7250
+F 0 "D8" H 5200 7350 50  0000 C CNN
+F 1 "LED" H 5200 7150 50  0000 C CNN
+F 2 "" H 5200 7250 50  0000 C CNN
+F 3 "" H 5200 7250 50  0000 C CNN
+	1    5200 7250
+	1    0    0    -1
+$EndComp
+$Comp
+L R R14
+U 1 1 59EA3DF3
+P 5700 5750
+F 0 "R14" V 5780 5750 50  0000 C CNN
+F 1 "300" V 5700 5750 50  0000 C CNN
+F 2 "Resistors_SMD:R_0603_HandSoldering" V 5630 5750 50  0001 C CNN
+F 3 "" H 5700 5750 50  0000 C CNN
+	1    5700 5750
+	0    -1   -1   0
+$EndComp
+$Comp
+L R R15
+U 1 1 59EA41C6
+P 5700 6050
+F 0 "R15" V 5780 6050 50  0000 C CNN
+F 1 "300" V 5700 6050 50  0000 C CNN
+F 2 "Resistors_SMD:R_0603_HandSoldering" V 5630 6050 50  0001 C CNN
+F 3 "" H 5700 6050 50  0000 C CNN
+	1    5700 6050
+	0    -1   -1   0
+$EndComp
+$Comp
+L R R16
+U 1 1 59EA4232
+P 5700 6350
+F 0 "R16" V 5780 6350 50  0000 C CNN
+F 1 "300" V 5700 6350 50  0000 C CNN
+F 2 "Resistors_SMD:R_0603_HandSoldering" V 5630 6350 50  0001 C CNN
+F 3 "" H 5700 6350 50  0000 C CNN
+	1    5700 6350
+	0    -1   -1   0
+$EndComp
+$Comp
+L R R17
+U 1 1 59EA4238
+P 5700 6650
+F 0 "R17" V 5780 6650 50  0000 C CNN
+F 1 "300" V 5700 6650 50  0000 C CNN
+F 2 "Resistors_SMD:R_0603_HandSoldering" V 5630 6650 50  0001 C CNN
+F 3 "" H 5700 6650 50  0000 C CNN
+	1    5700 6650
+	0    -1   -1   0
+$EndComp
+$Comp
+L R R18
+U 1 1 59EA4414
+P 5700 6950
+F 0 "R18" V 5780 6950 50  0000 C CNN
+F 1 "300" V 5700 6950 50  0000 C CNN
+F 2 "Resistors_SMD:R_0603_HandSoldering" V 5630 6950 50  0001 C CNN
+F 3 "" H 5700 6950 50  0000 C CNN
+	1    5700 6950
+	0    -1   -1   0
+$EndComp
+$Comp
+L R R19
+U 1 1 59EA441A
+P 5700 7250
+F 0 "R19" V 5780 7250 50  0000 C CNN
+F 1 "300" V 5700 7250 50  0000 C CNN
+F 2 "Resistors_SMD:R_0603_HandSoldering" V 5630 7250 50  0001 C CNN
+F 3 "" H 5700 7250 50  0000 C CNN
+	1    5700 7250
+	0    -1   -1   0
+$EndComp
+Wire Wire Line
+	5400 5750 5550 5750
+Wire Wire Line
+	5400 6050 5550 6050
+Wire Wire Line
+	5400 6350 5550 6350
+Wire Wire Line
+	5400 6650 5550 6650
+Wire Wire Line
+	5400 6950 5550 6950
+Wire Wire Line
+	5400 7250 5550 7250
+Wire Wire Line
+	5850 7250 6100 7250
+Wire Wire Line
+	6100 7250 6100 5500
+$Comp
+L +3.3V #PWR013
+U 1 1 59EA520A
+P 6100 5500
+F 0 "#PWR013" H 6100 5350 50  0001 C CNN
+F 1 "+3.3V" H 6100 5640 50  0000 C CNN
+F 2 "" H 6100 5500 50  0000 C CNN
+F 3 "" H 6100 5500 50  0000 C CNN
+	1    6100 5500
+	1    0    0    -1
+$EndComp
+Wire Wire Line
+	5850 5750 6100 5750
+Connection ~ 6100 5750
+Wire Wire Line
+	5850 6050 6100 6050
+Connection ~ 6100 6050
+Wire Wire Line
+	5850 6350 6100 6350
+Connection ~ 6100 6350
+Wire Wire Line
+	5850 6650 6100 6650
+Connection ~ 6100 6650
+Wire Wire Line
+	5850 6950 6100 6950
+Connection ~ 6100 6950
+Text GLabel 4800 5750 0    60   Input ~ 0
+led0
+Text GLabel 4800 6050 0    60   Input ~ 0
+led1
+Text GLabel 4800 6350 0    60   Input ~ 0
+led2
+Text GLabel 4800 6650 0    60   Input ~ 0
+led3
+Text GLabel 4800 6950 0    60   Input ~ 0
+led4
+Text GLabel 4800 7250 0    60   Input ~ 0
+led5
+Wire Wire Line
+	4800 7250 5000 7250
+Wire Wire Line
+	4800 6950 5000 6950
+Wire Wire Line
+	4800 6650 5000 6650
+Wire Wire Line
+	4800 6350 5000 6350
+Wire Wire Line
+	4800 6050 5000 6050
+Wire Wire Line
+	4800 5750 5000 5750
 $EndSCHEMATC

Commit message: change some pcb packages
Parts:
- D3, D4, D5, D6, D7, D8: footprint (none) -> LEDs:LED_0603
- R1, R14, R15, R16, R17, R18, R19, R3, R4, R5, R6, R7: footprint Resistors_SMD:R_0603_HandSoldering -> Resistors_SMD:R_0603
- R2: footprint Resistors_ThroughHole:R_Axial_DIN0207_L6.3mm_D2.5mm_P10.16mm_Horizontal -> Resistors_SMD:R_2512
Changed lines of the file:
@@
 F 0 "R1" V 980 2050 50  0000 C CNN
 F 1 "300" V 900 2050 50  0000 C CNN
-F 2 "Resistors_SMD:R_0603_HandSoldering" V 830 2050 50  0001 C CNN
+F 2 "Resistors_SMD:R_0603" V 830 2050 50  0001 C CNN
 F 3 "" H 900 2050 50  0000 C CNN
 	1    900  2050
@@
 F 0 "R3" V 2530 2050 50  0000 C CNN
 F 1 "300" V 2450 2050 50  0000 C CNN
-F 2 "Resistors_SMD:R_0603_HandSoldering" V 2380 2050 50  0001 C CNN
+F 2 "Resistors_SMD:R_0603" V 2380 2050 50  0001 C CNN
 F 3 "" H 2450 2050 50  0000 C CNN
 	1    2450 2050
@@
 F 0 "R4" V 4030 2050 50  0000 C CNN
 F 1 "300" V 3950 2050 50  0000 C CNN
-F 2 "Resistors_SMD:R_0603_HandSoldering" V 3880 2050 50  0001 C CNN
+F 2 "Resistors_SMD:R_0603" V 3880 2050 50  0001 C CNN
 F 3 "" H 3950 2050 50  0000 C CNN
 	1    3950 2050
@@
 F 0 "R5" V 5530 2050 50  0000 C CNN
 F 1 "300" V 5450 2050 50  0000 C CNN
-F 2 "Resistors_SMD:R_0603_HandSoldering" V 5380 2050 50  0001 C CNN
+F 2 "Resistors_SMD:R_0603" V 5380 2050 50  0001 C CNN
 F 3 "" H 5450 2050 50  0000 C CNN
 	1    5450 2050
@@
 F 0 "R6" V 7030 2050 50  0000 C CNN
 F 1 "300" V 6950 2050 50  0000 C CNN
-F 2 "Resistors_SMD:R_0603_HandSoldering" V 6880 2050 50  0001 C CNN
+F 2 "Resistors_SMD:R_0603" V 6880 2050 50  0001 C CNN
 F 3 "" H 6950 2050 50  0000 C CNN
 	1    6950 2050
@@
 F 0 "R7" V 8530 2050 50  0000 C CNN
 F 1 "300" V 8450 2050 50  0000 C CNN
-F 2 "Resistors_SMD:R_0603_HandSoldering" V 8380 2050 50  0001 C CNN
+F 2 "Resistors_SMD:R_0603" V 8380 2050 50  0001 C CNN
 F 3 "" H 8450 2050 50  0000 C CNN
 	1    8450 2050
@@
 F 0 "R2" V 1480 1000 50  0000 C CNN
 F 1 "20k" V 1400 1000 50  0000 C CNN
-F 2 "Resistors_ThroughHole:R_Axial_DIN0207_L6.3mm_D2.5mm_P10.16mm_Horizontal" V 1330 1000 50  0001 C CNN
+F 2 "Resistors_SMD:R_2512" V 1330 1000 50  0001 C CNN
 F 3 "" H 1400 1000 50  0000 C CNN
 	1    1400 1000
@@
 F 0 "D3" H 5200 5850 50  0000 C CNN
 F 1 "LED" H 5200 5650 50  0000 C CNN
-F 2 "" H 5200 5750 50  0000 C CNN
+F 2 "LEDs:LED_0603" H 5200 5750 50  0001 C CNN
 F 3 "" H 5200 5750 50  0000 C CNN
 	1    5200 5750
@@
 F 0 "D4" H 5200 6150 50  0000 C CNN
 F 1 "LED" H 5200 5950 50  0000 C CNN
-F 2 "" H 5200 6050 50  0000 C CNN
+F 2 "LEDs:LED_0603" H 5200 6050 50  0001 C CNN
 F 3 "" H 5200 6050 50  0000 C CNN
 	1    5200 6050
@@
 F 0 "D5" H 5200 6450 50  0000 C CNN
 F 1 "LED" H 5200 6250 50  0000 C CNN
-F 2 "" H 5200 6350 50  0000 C CNN
+F 2 "LEDs:LED_0603" H 5200 6350 50  0001 C CNN
 F 3 "" H 5200 6350 50  0000 C CNN
 	1    5200 6350
@@
 F 0 "D6" H 5200 6750 50  0000 C CNN
 F 1 "LED" H 5200 6550 50  0000 C CNN
-F 2 "" H 5200 6650 50  0000 C CNN
+F 2 "LEDs:LED_0603" H 5200 6650 50  0001 C CNN
 F 3 "" H 5200 6650 50  0000 C CNN
 	1    5200 6650
@@
 F 0 "D7" H 5200 7050 50  0000 C CNN
 F 1 "LED" H 5200 6850 50  0000 C CNN
-F 2 "" H 5200 6950 50  0000 C CNN
+F 2 "LEDs:LED_0603" H 5200 6950 50  0001 C CNN
 F 3 "" H 5200 6950 50  0000 C CNN
 	1    5200 6950
@@
 F 0 "D8" H 5200 7350 50  0000 C CNN
 F 1 "LED" H 5200 7150 50  0000 C CNN
-F 2 "" H 5200 7250 50  0000 C CNN
+F 2 "LEDs:LED_0603" H 5200 7250 50  0001 C CNN
 F 3 "" H 5200 7250 50  0000 C CNN
 	1    5200 7250
@@
 F 0 "R14" V 5780 5750 50  0000 C CNN
 F 1 "300" V 5700 5750 50  0000 C CNN
-F 2 "Resistors_SMD:R_0603_HandSoldering" V 5630 5750 50  0001 C CNN
+F 2 "Resistors_SMD:R_0603" V 5630 5750 50  0001 C CNN
 F 3 "" H 5700 5750 50  0000 C CNN
 	1    5700 5750
@@
 F 0 "R15" V 5780 6050 50  0000 C CNN
 F 1 "300" V 5700 6050 50  0000 C CNN
-F 2 "Resistors_SMD:R_0603_HandSoldering" V 5630 6050 50  0001 C CNN
+F 2 "Resistors_SMD:R_0603" V 5630 6050 50  0001 C CNN
 F 3 "" H 5700 6050 50  0000 C CNN
 	1    5700 6050
@@
 F 0 "R16" V 5780 6350 50  0000 C CNN
 F 1 "300" V 5700 6350 50  0000 C CNN
-F 2 "Resistors_SMD:R_0603_HandSoldering" V 5630 6350 50  0001 C CNN
+F 2 "Resistors_SMD:R_0603" V 5630 6350 50  0001 C CNN
 F 3 "" H 5700 6350 50  0000 C CNN
 	1    5700 6350
@@
 F 0 "R17" V 5780 6650 50  0000 C CNN
 F 1 "300" V 5700 6650 50  0000 C CNN
-F 2 "Resistors_SMD:R_0603_HandSoldering" V 5630 6650 50  0001 C CNN
+F 2 "Resistors_SMD:R_0603" V 5630 6650 50  0001 C CNN
 F 3 "" H 5700 6650 50  0000 C CNN
 	1    5700 6650
@@
 F 0 "R18" V 5780 6950 50  0000 C CNN
 F 1 "300" V 5700 6950 50  0000 C CNN
-F 2 "Resistors_SMD:R_0603_HandSoldering" V 5630 6950 50  0001 C CNN
+F 2 "Resistors_SMD:R_0603" V 5630 6950 50  0001 C CNN
 F 3 "" H 5700 6950 50  0000 C CNN
 	1    5700 6950
@@
 F 0 "R19" V 5780 7250 50  0000 C CNN
 F 1 "300" V 5700 7250 50  0000 C CNN
-F 2 "Resistors_SMD:R_0603_HandSoldering" V 5630 7250 50  0001 C CNN
+F 2 "Resistors_SMD:R_0603" V 5630 7250 50  0001 C CNN
 F 3 "" H 5700 7250 50  0000 C CNN
 	1    5700 7250

Commit message: many changes
Parts:
- added NT10, NT7, NT8, NT9: IN-3, nixie_clock:IN-3, symbol IN-3
- added R1, R3, R4, R5, R6: 20k, Resistors_SMD:R_2512, symbol R
- added R19, R20, R22: 300, Resistors_SMD:R_0603, symbol R
- added R21, R23: 100k, Resistors_SMD:R_2512, symbol R
- added U6: TLP627, Housings_DIP:DIP-4_W7.62mm, symbol TLP627
- added U7: TLP627-2, Housings_DIP:DIP-8_W7.62mm, symbol TLP627-2
- renumbered D3 to D1, D4 to D2, D5 to D3, D6 to D4, D7 to D5, D8 to D6, R5 to R10, R6 to R11, R7 to R12, R14 to R13, R15 to R14, R16 to R15, R17 to R16, R18 to R17, R19 to R18, R1 to R7, R3 to R8, R4 to R9, U4 to U3, U5 to U4, U3 to U5
Connections:
- net +3V3: now also R19.1, R20.1, R22.1
- net GND: now also NT7.2, NT9.2, U6.3
- net VNXE: now also R2.1, R1.1, R21.1, R23.1, R3.1, R4.1, R5.1, R6.1; no longer R2.2
- net at NT1.12 (dot): now also NT2.12 (dot), NT3.12 (dot), NT4.12 (dot), NT5.12 (dot), NT6.12 (dot), U6.4
- new net: R1.2, U2.8
- new net: R2.2, U2.6
- new net: R3.2, U3.8
- new net: R4.2, U3.6
- new net: R5.2, U4.8
- new net: R6.2, U4.6
- new net: R20.2, U7.1
- new net: NT8.1, U7.7
- new net: R21.2, U7.8
- new net: R22.2, U7.3
- new net: NT10.1, U7.5
- new net: R23.2, U7.6
- new net: R19.2, U6.1
- new net: NT7.1, NT8.2
- new net: NT10.2, NT9.1
- new net nxecol0: U7.2
- new net nxecol1: U7.4
- new net nxedot: U6.2
- no-connect marks 6 -> 0
Other:
- note added: "1/2W"
- moved on the sheet: D1, D2, D3, D4, D5, D6, NT1, NT2, NT3, NT4, NT5, NT6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

Commit message: add connectors
Parts:
- added P1, P2, P3, P4: CONN_02X05, Socket_Strips:Socket_Strip_Straight_2x05_Pitch2.54mm, symbol CONN_02X05
- NT10, NT7, NT8, NT9: footprint nixie_clock:IN-3 -> (none)
Connections:
- net nc0: now reaches NT1.1 (COM)
- net nc0: now also P3.1 (P1); no longer U2.7
- net n2: now reaches NT1.10 (2), NT2.10 (2), NT3.10 (2), NT4.10 (2), NT5.10 (2), NT6.10 (2)
- net n2: now also P1.3 (P3); no longer U5.8 (2)
- net n1: now reaches NT1.11 (1), NT2.11 (1), NT3.11 (1), NT4.11 (1), NT5.11 (1), NT6.11 (1)
- net n1: now also P1.1 (P1); no longer U5.15 (1)
- net ndot: now reaches NT1.12 (dot), NT2.12 (dot), NT3.12 (dot), NT4.12 (dot), NT5.12 (dot), NT6.12 (dot)
- net ndot: now also P3.6 (P6); no longer U6.4
- net n0: now reaches NT1.2 (0), NT2.2 (0), NT3.2 (0), NT4.2 (0), NT5.2 (0), NT6.2 (0)
- net n0: now also P1.10 (P10); no longer U5.16 (0)
- net n9: now reaches NT1.3 (9), NT2.3 (9), NT3.3 (9), NT4.3 (9), NT5.3 (9), NT6.3 (9)
- net n9: now also P1.8 (P8); no longer U5.2 (9)
- net n8: now reaches NT1.4 (8), NT2.4 (8), NT3.4 (8), NT4.4 (8), NT5.4 (8), NT6.4 (8)
- net n8: now also P1.6 (P6); no longer U5.1 (8)
- net n7: now reaches NT1.5 (7), NT2.5 (7), NT3.5 (7), NT4.5 (7), NT5.5 (7), NT6.5 (7)
- net n7: now also P1.4 (P4); no longer U5.10 (7)
- net n6: now reaches NT1.6, NT2.6, NT3.6, NT4.6, NT5.6, NT6.6
- net n6: now also P1.2 (P2); no longer U5.11 (6)
- net n5: now reaches NT1.7 (5), NT2.7 (5), NT3.7 (5), NT4.7 (5), NT5.7 (5), NT6.7 (5)
- net n5: now also P1.9 (P9); no longer U5.14 (5)
- net n4: now reaches NT1.8 (4), NT2.8 (4), NT3.8 (4), NT4.8 (4), NT5.8 (4), NT6.8 (4)
- net n4: now also P1.7 (P7); no longer U5.13 (4)
- net n3: now reaches NT1.9 (3), NT2.9 (3), NT3.9 (3), NT4.9 (3), NT5.9 (3), NT6.9 (3)
- net n3: now also P1.5 (P5); no longer U5.9 (3)
- net nc1: now reaches NT2.1 (COM)
- net nc1: now also P3.3 (P3); no longer U2.5
- net nc2: now reaches NT3.1 (COM)
- net nc2: now also P3.5 (P5); no longer U3.7
- net nc3: now reaches NT4.1 (COM)
- net nc3: now also P3.7 (P7); no longer U3.5
- net nc4: now reaches NT5.1 (COM)
- net nc4: now also P3.9 (P9); no longer U4.7
- net nc5: now reaches NT6.1 (COM)
- net nc5: now also P3.10 (P10); no longer U4.5
- net ncol0: now reaches NT8.1
- net ncol0: now also P3.4 (P4); no longer U7.7
- net ncol1: now reaches NT10.1
- net ncol1: now also P3.2 (P2); no longer U7.5
- new net nm0: P2.10 (P10), U5.16 (0)
- new net nm1: P2.1 (P1), U5.15 (1)
- new net nm2: P2.3 (P3), U5.8 (2)
- new net nm3: P2.5 (P5), U5.9 (3)
- new net nm4: P2.7 (P7), U5.13 (4)
- new net nm5: P2.9 (P9), U5.14 (5)
- new net nm6: P2.2 (P2), U5.11 (6)
- new net nm7: P2.4 (P4), U5.10 (7)
- new net nm8: P2.6 (P6), U5.1 (8)
- new net nm9: P2.8 (P8), U5.2 (9)
- new net nmc0: P4.1 (P1), U2.7
- new net nmc1: P4.3 (P3), U2.5
- new net nmc2: P4.5 (P5), U3.7
- new net nmc3: P4.7 (P7), U3.5
- new net nmc4: P4.9 (P9), U4.7
- new net nmc5: P4.10 (P10), U4.5
- new net nmcol0: P4.4 (P4), U7.7
- new net nmcol1: P4.2 (P2), U7.5
- new net nmdot: P4.6 (P6), U6.4
- no-connect marks 0 -> 2
Other:
- moved on the sheet: R1, R10, R11, R12, R2, R3, R4, R5, R6, R7, R8, R9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
