File: KiCad/nixie.sch (KiCad schematic (older format))
At the start: 49 parts, among them P1 CONN_02X05, P2 CONN_02X05, P3 CONN_02X05, P4 CONN_02X05, U2 TLP627-2, U3 TLP627-2, U4 TLP627-2, U5 SN74141, U6 TLP627, U7 TLP627-2

Commit message: add edge cuts
Parts:
- NT10, NT7, NT8, NT9: footprint (none) -> nixie_clock:IN-3
Connections:
- net GND: no longer NT7.2, NT9.2
- net n0: now also P1.2 (P2); no longer P1.10 (P10)
- net n6: now also P1.10 (P10); no longer P1.2 (P2)
- net n7: now also P1.8 (P8); no longer P1.4 (P4)
- net n9: now also P1.4 (P4); no longer P1.8 (P8)
- net nc0: now also P3.9 (P9); no longer P3.1 (P1)
- net nc1: now also P3.7 (P7); no longer P3.3 (P3)
- net nc3: now also P3.3 (P3); no longer P3.7 (P7)
- net nc4: now also P3.1 (P1); no longer P3.9 (P9)
- net nc5: now also P3.2 (P2); no longer P3.10 (P10)
- net ncol0: now also P3.8 (P8); no longer P3.4 (P4)
- net ncol1: now also P3.6 (P6); no longer P3.2 (P2)
- net ndot: now also P3.4 (P4); no longer P3.6 (P6)
- net nm0: now also P2.2 (P2); no longer P2.10 (P10)
- net nm6: now also P2.10 (P10); no longer P2.2 (P2)
- net nm7: now also P2.8 (P8); no longer P2.4 (P4)
- net nm9: now also P2.4 (P4); no longer P2.8 (P8)
- net nmc0: now also P4.9 (P9); no longer P4.1 (P1)
- net nmc1: now also P4.7 (P7); no longer P4.3 (P3)
- net nmc3: now also P4.3 (P3); no longer P4.7 (P7)
- net nmc4: now also P4.1 (P1); no longer P4.9 (P9)
- net nmc5: now also P4.2 (P2); no longer P4.10 (P10)
- net nmcol0: now also P4.8 (P8); no longer P4.4 (P4)
- net nmcol1: now also P4.6 (P6); no longer P4.2 (P2)
- net nmdot: now also P4.4 (P4); no longer P4.6 (P6)
- new net ngnd: NT7.2, NT9.2, P3.10 (P10)
- new net nmgnd: P4.10 (P10)
- no-connect marks 2 -> 0
Changed lines of the file:
@@
-	1    0    0    -1
-$EndComp
-$Comp
-L GND #PWR016
-U 1 1 59EF503E
-P 4450 7400
-F 0 "#PWR016" H 4450 7150 50  0001 C CNN
-F 1 "GND" H 4450 7250 50  0000 C CNN
-F 2 "" H 4450 7400 50  0000 C CNN
-F 3 "" H 4450 7400 50  0000 C CNN
-	1    4450 7400
-	1    0    0    -1
-$EndComp
-$Comp
-L GND #PWR017
-U 1 1 59EF5152
-P 5850 7400
-F 0 "#PWR017" H 5850 7150 50  0001 C CNN
-F 1 "GND" H 5850 7250 50  0000 C CNN
-F 2 "" H 5850 7400 50  0000 C CNN
-F 3 "" H 5850 7400 50  0000 C CNN
-	1    5850 7400
 	1    0    0    -1
 $EndComp
@@
 VNXE
 $Comp
-L +3.3V #PWR018
+L +3.3V #PWR016
 U 1 1 59EFD3BA
 P 4400 5250
-F 0 "#PWR018" H 4400 5100 50  0001 C CNN
+F 0 "#PWR016" H 4400 5100 50  0001 C CNN
 F 1 "+3.3V" H 4400 5390 50  0000 C CNN
 F 2 "" H 4400 5250 50  0000 C CNN
@@
 $EndComp
 $Comp
-L +3.3V #PWR019
+L +3.3V #PWR017
 U 1 1 59EFDEAE
 P 6050 5250
-F 0 "#PWR019" H 6050 5100 50  0001 C CNN
+F 0 "#PWR017" H 6050 5100 50  0001 C CNN
 F 1 "+3.3V" H 6050 5390 50  0000 C CNN
 F 2 "" H 6050 5250 50  0000 C CNN
@@
 Text Label 650  4150 3    60   ~ 0
 n5
-Text Label 1050 5150 1    60   ~ 0
+Text Label 650  5150 1    60   ~ 0
 n6
-Text Label 950  5150 1    60   ~ 0
+Text Label 750  5150 1    60   ~ 0
 n7
 Text Label 850  5150 1    60   ~ 0
 n8
-Text Label 750  5150 1    60   ~ 0
+Text Label 950  5150 1    60   ~ 0
 n9
-Text Label 650  5150 1    60   ~ 0
+Text Label 1050 5150 1    60   ~ 0
 n0
 Text Label 1050 5300 3    60   ~ 0
@@
 Text Label 650  5300 3    60   ~ 0
 nm5
-Text Label 1050 6300 1    60   ~ 0
+Text Label 650  6300 1    60   ~ 0
 nm6
-Text Label 950  6300 1    60   ~ 0
+Text Label 750  6300 1    60   ~ 0
 nm7
 Text Label 850  6300 1    60   ~ 0
 nm8
-Text Label 750  6300 1    60   ~ 0
+Text Label 950  6300 1    60   ~ 0
 nm9
-Text Label 650  6300 1    60   ~ 0
+Text Label 1050 6300 1    60   ~ 0
 nm0
 $Comp
@@
 Text Label 9350 2850 3    60   ~ 0
 nc5
-Text Label 10800 3650 3    60   ~ 0
+Text Label 10400 3650 3    60   ~ 0
 nc0
-Text Label 10700 3650 3    60   ~ 0
+Text Label 10500 3650 3    60   ~ 0
 nc1
 Text Label 10600 3650 3    60   ~ 0
 nc2
-Text Label 10500 3650 3    60   ~ 0
+Text Label 10700 3650 3    60   ~ 0
 nc3
-Text Label 10400 3650 3    60   ~ 0
+Text Label 10800 3650 3    60   ~ 0
 nc4
-Text Label 10400 4850 1    60   ~ 0
+Text Label 10800 4850 1    60   ~ 0
 nc5
-Text Label 10400 6300 1    60   ~ 0
+Text Label 10800 6300 1    60   ~ 0
 nmc5
-Text Label 10400 5100 3    60   ~ 0
+Text Label 10800 5100 3    60   ~ 0
 nmc4
-Text Label 10500 5100 3    60   ~ 0
+Text Label 10700 5100 3    60   ~ 0
 nmc3
 Text Label 10600 5100 3    60   ~ 0
 nmc2
-Text Label 10700 5100 3    60   ~ 0
+Text Label 10500 5100 3    60   ~ 0
 nmc1
-Text Label 10800 5100 3    60   ~ 0
+Text Label 10400 5100 3    60   ~ 0
 nmc0
 Wire Wire Line
@@
 Text Label 3850 5500 3    60   ~ 0
 nmdot
-Text Label 10600 4850 1    60   ~ 0
+Text Label 10700 4850 1    60   ~ 0
 ndot
-Text Label 10600 6300 1    60   ~ 0
+Text Label 10700 6300 1    60   ~ 0
 nmdot
 Text Label 5550 6050 2    60   ~ 0
@@
 Text Label 7000 6400 2    60   ~ 0
 ncol1
-Text Label 10700 6300 1    60   ~ 0
+Text Label 10500 6300 1    60   ~ 0
 nmcol0
-Text Label 10800 6300 1    60   ~ 0
+Text Label 10600 6300 1    60   ~ 0
 nmcol1
-Text Label 10700 4850 1    60   ~ 0
+Text Label 10500 4850 1    60   ~ 0
 ncol0
-Text Label 10800 4850 1    60   ~ 0
+Text Label 10600 4850 1    60   ~ 0
 ncol1
-NoConn ~ 10500 4850
-NoConn ~ 10500 6300
 $Comp
 L IN-3 NT7
@@
 F 0 "NT7" V 4230 6720 60  0000 C CNN
 F 1 "IN-3" V 4150 6730 60  0000 C CNN
-F 2 "" H 4450 6750 60  0000 C CNN
+F 2 "nixie_clock:IN-3" H 4450 6750 60  0001 C CNN
 F 3 "" H 4450 6750 60  0000 C CNN
 	1    4450 6750
@@
 F 0 "NT8" V 4780 6720 60  0000 C CNN
 F 1 "IN-3" V 4700 6730 60  0000 C CNN
-F 2 "" H 5000 6750 60  0000 C CNN
+F 2 "nixie_clock:IN-3" H 5000 6750 60  0001 C CNN
 F 3 "" H 5000 6750 60  0000 C CNN
 	1    5000 6750
@@
 F 0 "NT9" V 5630 6720 60  0000 C CNN
 F 1 "IN-3" V 5550 6730 60  0000 C CNN
-F 2 "" H 5850 6750 60  0000 C CNN
+F 2 "nixie_clock:IN-3" H 5850 6750 60  0001 C CNN
 F 3 "" H 5850 6750 60  0000 C CNN
 	1    5850 6750
@@
 F 0 "NT10" V 6180 6720 60  0000 C CNN
 F 1 "IN-3" V 6100 6730 60  0000 C CNN
-F 2 "" H 6400 6750 60  0000 C CNN
+F 2 "nixie_clock:IN-3" H 6400 6750 60  0001 C CNN
 F 3 "" H 6400 6750 60  0000 C CNN
 	1    6400 6750
 	1    0    0    -1
 $EndComp
+Text Label 10400 4850 1    60   ~ 0
+ngnd
+Text Label 10400 6300 1    60   ~ 0
+nmgnd
+Text Label 5850 7400 1    60   ~ 0
+ngnd
+Text Label 4450 7400 1    60   ~ 0
+ngnd
 $EndSCHEMATC
