File: KiCad/nixie.sch (KiCad schematic (older format))
At the start: 49 parts, among them P1 CONN_02X05, P2 CONN_02X05, P3 CONN_02X05, P4 CONN_02X05, U2 TLP627-2, U3 TLP627-2, U4 TLP627-2, U5 SN74141, U6 TLP627, U7 TLP627-2

Commit message: change pcb designs
Connections:
- net nmgnd is gone; now on net GND: P4.10 (P10)
- net n2: now also P1.8 (P8); no longer P1.3 (P3)
- net n3: now also P1.10 (P10); no longer P1.5 (P5)
- net n4: now also P1.5 (P5); no longer P1.7 (P7)
- net n5: now also P1.3 (P3); no longer P1.9 (P9)
- net n6: now also P1.7 (P7); no longer P1.10 (P10)
- net n7: now also P1.9 (P9); no longer P1.8 (P8)
- net n8: now also P1.4 (P4); no longer P1.6 (P6)
- net n9: now also P1.6 (P6); no longer P1.4 (P4)
- net nm2: now also P2.8 (P8); no longer P2.3 (P3)
- net nm3: now also P2.10 (P10); no longer P2.5 (P5)
- net nm4: now also P2.5 (P5); no longer P2.7 (P7)
- net nm5: now also P2.3 (P3); no longer P2.9 (P9)
- net nm6: now also P2.7 (P7); no longer P2.10 (P10)
- net nm7: now also P2.9 (P9); no longer P2.8 (P8)
- net nm8: now also P2.4 (P4); no longer P2.6 (P6)
- net nm9: now also P2.6 (P6); no longer P2.4 (P4)
Changed lines of the file:
@@
 Text Label 1050 4150 3    60   ~ 0
 n1
+Text Label 750  5150 1    60   ~ 0
+n2
+Text Label 650  5150 1    60   ~ 0
+n3
+Text Label 850  4150 3    60   ~ 0
+n4
 Text Label 950  4150 3    60   ~ 0
-n2
-Text Label 850  4150 3    60   ~ 0
-n3
+n5
 Text Label 750  4150 3    60   ~ 0
-n4
+n6
 Text Label 650  4150 3    60   ~ 0
-n5
-Text Label 650  5150 1    60   ~ 0
-n6
-Text Label 750  5150 1    60   ~ 0
 n7
+Text Label 950  5150 1    60   ~ 0
+n8
 Text Label 850  5150 1    60   ~ 0
-n8
-Text Label 950  5150 1    60   ~ 0
 n9
 Text Label 1050 5150 1    60   ~ 0
@@
 Text Label 1050 5300 3    60   ~ 0
 nm1
+Text Label 750  6300 1    60   ~ 0
+nm2
+Text Label 650  6300 1    60   ~ 0
+nm3
+Text Label 850  5300 3    60   ~ 0
+nm4
 Text Label 950  5300 3    60   ~ 0
-nm2
-Text Label 850  5300 3    60   ~ 0
-nm3
+nm5
 Text Label 750  5300 3    60   ~ 0
-nm4
+nm6
 Text Label 650  5300 3    60   ~ 0
-nm5
-Text Label 650  6300 1    60   ~ 0
-nm6
-Text Label 750  6300 1    60   ~ 0
 nm7
+Text Label 950  6300 1    60   ~ 0
+nm8
 Text Label 850  6300 1    60   ~ 0
-nm8
-Text Label 950  6300 1    60   ~ 0
 nm9
 Text Label 1050 6300 1    60   ~ 0
@@
 Text Label 4450 7400 1    60   ~ 0
 ngnd
+$Comp
+L GND #PWR018
+U 1 1 59F225AA
+P 10400 6300
+F 0 "#PWR018" H 10400 6050 50  0001 C CNN
+F 1 "GND" H 10400 6150 50  0000 C CNN
+F 2 "" H 10400 6300 50  0000 C CNN
+F 3 "" H 10400 6300 50  0000 C CNN
+	1    10400 6300
+	1    0    0    -1
+$EndComp
 $EndSCHEMATC

Commit message: finish route
Connections:
- net nmc0: now also U2.5; no longer U2.7
- net nmc1: now also U2.7; no longer U2.5
- net nmc4: now also U4.5; no longer U4.7
- net nmc5: now also U4.7; no longer U4.5
- net nxecom0: now also U2.4; no longer U2.2
- net nxecom1: now also U2.2; no longer U2.4
- net nxecom4: now also U4.4; no longer U4.2
- net nxecom5: now also U4.2; no longer U4.4
- net at R7.2: now also U2.3; no longer U2.1
- net at R1.2: now also U2.6; no longer U2.8
- net at R8.2: now also U2.1; no longer U2.3
- net at R2.2: now also U2.8; no longer U2.6
- net at R11.2: now also U4.3; no longer U4.1
- net at R5.2: now also U4.6; no longer U4.8
- net at R12.2: now also U4.1; no longer U4.3
- net at R6.2: now also U4.8; no longer U4.6
Changed lines of the file:
@@
 $Comp
 L TLP627-2 U2
-U 1 1 59E2402B
+U 2 1 59E2402B
 P 1450 2150
 F 0 "U2" H 1150 2350 50  0000 L CNN
@@
 F 2 "Housings_DIP:DIP-8_W7.62mm" H 1150 1950 50  0001 L CIN
 F 3 "" H 1450 2150 50  0000 L CNN
-	1    1450 2150
+	2    1450 2150
 	1    0    0    -1
 $EndComp
 $Comp
 L TLP627-2 U2
-U 2 1 59E24124
+U 1 1 59E24124
 P 2950 2150
 F 0 "U2" H 2650 2350 50  0000 L CNN
@@
 F 2 "Housings_DIP:DIP-8_W7.62mm" H 2650 1950 50  0001 L CIN
 F 3 "" H 2950 2150 50  0000 L CNN
-	2    2950 2150
+	1    2950 2150
 	1    0    0    -1
 $EndComp
@@
 $Comp
 L TLP627-2 U4
-U 1 1 59E24315
+U 2 1 59E24315
 P 7450 2150
 F 0 "U4" H 7150 2350 50  0000 L CNN
@@
 F 2 "Housings_DIP:DIP-8_W7.62mm" H 7150 1950 50  0001 L CIN
 F 3 "" H 7450 2150 50  0000 L CNN
-	1    7450 2150
+	2    7450 2150
 	1    0    0    -1
 $EndComp
 $Comp
 L TLP627-2 U4
-U 2 1 59E2431B
+U 1 1 59E2431B
 P 8950 2150
 F 0 "U4" H 8650 2350 50  0000 L CNN
@@
 F 2 "Housings_DIP:DIP-8_W7.62mm" H 8650 1950 50  0001 L CIN
 F 3 "" H 8950 2150 50  0000 L CNN
-	2    8950 2150
+	1    8950 2150
 	1    0    0    -1
 $EndComp
