File: KiCad/power.sch (KiCad schematic (older format))
At the start: 22 parts, among them CON1 BARREL_JACK, Q1 2SA1015, Q2 2SK3234, U6 NJM2360A, U7 NJM7805S

Commit message: many changes
Parts:
- renumbered C7 to C2, C2 to C4, C4 to C5, C5 to C6, C6 to C7, D2 to D7, D1 to D8, Q2 to Q1, Q1 to Q2, R8 to R24, R9 to R25, R10 to R26, R12 to R27, R13 to R28, R11 to R29, U6 to U8, U7 to U9
Changed lines of the file:
@@
 Sheet 4 4
 Title "power"
-Date "2017-10-16"
+Date "2017-10-24"
 Rev ""
 Comp ""
@@
 $EndDescr
 $Comp
-L NJM2360A U6
+L NJM2360A U8
 U 1 1 59E34B10
 P 3650 2100
-F 0 "U6" H 3650 2350 60  0000 C CNN
+F 0 "U8" H 3650 2350 60  0000 C CNN
 F 1 "NJM2360A" H 3650 1850 60  0000 C CNN
 F 2 "Housings_DIP:DIP-8_W7.62mm" H 3400 2100 60  0001 C CNN
@@
 $EndComp
 $Comp
-L 2SA1016 Q1
+L 2SA1016 Q2
 U 1 1 59E35C01
 P 5550 2350
-F 0 "Q1" H 5750 2425 50  0000 L CNN
+F 0 "Q2" H 5750 2425 50  0000 L CNN
 F 1 "2SA1015" H 5750 2350 50  0000 L CNN
 F 2 "TO_SOT_Packages_THT:TO-92_Inline_Wide" H 5750 2275 50  0001 L CIN
@@
 $EndComp
 $Comp
-L Q_NMOS_GDS Q2
+L Q_NMOS_GDS Q1
 U 1 1 59E35CC2
 P 6050 1950
-F 0 "Q2" H 6350 2000 50  0000 R CNN
+F 0 "Q1" H 6350 2000 50  0000 R CNN
 F 1 "2SK3234" H 6600 1900 50  0000 R CNN
 F 2 "TO_SOT_Packages_THT:TO-220-3_Vertical" H 6250 2050 50  0001 C CNN
@@
 $EndComp
 $Comp
-L D_Schottky D2
+L D_Schottky D7
 U 1 1 59E35CF9
 P 6700 1400
-F 0 "D2" H 6700 1500 50  0000 C CNN
+F 0 "D7" H 6700 1500 50  0000 C CNN
 F 1 "UF2010" H 6700 1300 50  0000 C CNN
 F 2 "Diodes_ThroughHole:D_A-405_P10.16mm_Horizontal" H 6700 1400 50  0001 C CNN
@@
 $EndComp
 $Comp
-L D D1
+L D D8
 U 1 1 59E35D4E
 P 5300 1950
-F 0 "D1" H 5300 2050 50  0000 C CNN
+F 0 "D8" H 5300 2050 50  0000 C CNN
 F 1 "1N4148W" H 5300 1850 50  0000 C CNN
 F 2 "Diodes_SMD:D_SOD-123" H 5300 1950 50  0001 C CNN
@@
 $EndComp
 $Comp
-L GND #PWR014
+L GND #PWR020
 U 1 1 59E35E0E
 P 6150 2950
-F 0 "#PWR014" H 6150 2700 50  0001 C CNN
+F 0 "#PWR020" H 6150 2700 50  0001 C CNN
 F 1 "GND" H 6150 2800 50  0000 C CNN
 F 2 "" H 6150 2950 50  0000 C CNN
@@
 $EndComp
 $Comp
-L R R11
+L R R29
 U 1 1 59E35E42
 P 5000 2700
-F 0 "R11" V 5080 2700 50  0000 C CNN
+F 0 "R29" V 5080 2700 50  0000 C CNN
 F 1 "1k" V 5000 2700 50  0000 C CNN
 F 2 "Resistors_SMD:R_1206" V 4930 2700 50  0001 C CNN
@@
 $EndComp
 $Comp
-L GND #PWR015
+L GND #PWR021
 U 1 1 59E35F44
 P 5000 2950
-F 0 "#PWR015" H 5000 2700 50  0001 C CNN
+F 0 "#PWR021" H 5000 2700 50  0001 C CNN
 F 1 "GND" H 5000 2800 50  0000 C CNN
 F 2 "" H 5000 2950 50  0000 C CNN
@@
 $EndComp
 $Comp
-L R R10
+L R R26
 U 1 1 59E3604C
 P 4200 1650
-F 0 "R10" V 4280 1650 50  0000 C CNN
+F 0 "R26" V 4280 1650 50  0000 C CNN
 F 1 "470" V 4200 1650 50  0000 C CNN
 F 2 "Resistors_SMD:R_1206" V 4130 1650 50  0001 C CNN
@@
 $EndComp
 $Comp
-L R R9
+L R R25
 U 1 1 59E36083
 P 3100 1650
-F 0 "R9" V 3180 1650 50  0000 C CNN
+F 0 "R25" V 3180 1650 50  0000 C CNN
 F 1 "1k" V 3100 1650 50  0000 C CNN
 F 2 "Resistors_SMD:R_1206" V 3030 1650 50  0001 C CNN
@@
 $EndComp
 $Comp
-L R R8
+L R R24
 U 1 1 59E3610B
 P 2650 1400
-F 0 "R8" V 2730 1400 50  0000 C CNN
+F 0 "R24" V 2730 1400 50  0000 C CNN
 F 1 "1" V 2650 1400 50  0000 C CNN
 F 2 "Resistors_SMD:R_2512" V 2580 1400 50  0001 C CNN
@@
 $EndComp
 $Comp
-L R R12
+L R R27
 U 1 1 59E36277
 P 7250 1750
-F 0 "R12" V 7330 1750 50  0000 C CNN
+F 0 "R27" V 7330 1750 50  0000 C CNN
 F 1 "470k" V 7250 1750 50  0000 C CNN
 F 2 "Resistors_SMD:R_1206" V 7180 1750 50  0001 C CNN
@@
 $EndComp
 $Comp
-L CP1 C7
+L CP1 C2
 U 1 1 59E36592
 P 7900 1750
-F 0 "C7" H 7925 1850 50  0000 L CNN
+F 0 "C2" H 7925 1850 50  0000 L CNN
 F 1 "10u/400V" H 7925 1650 50  0000 L CNN
 F 2 "Capacitors_ThroughHole:CP_Radial_D12.5mm_P5.00mm" H 7900 1750 50  0001 C CNN
@@
 Connection ~ 7250 1400
 $Comp
-L R R13
+L R R28
 U 1 1 59E36938
 P 7250 2650
-F 0 "R13" V 7330 2650 50  0000 C CNN
+F 0 "R28" V 7330 2650 50  0000 C CNN
 F 1 "470" V 7250 2650 50  0000 C CNN
 F 2 "Resistors_SMD:R_1206" V 7180 2650 50  0001 C CNN
@@
 $EndComp
 $Comp
-L GND #PWR016
+L GND #PWR022
 U 1 1 59E3695E
 P 7250 2950
-F 0 "#PWR016" H 7250 2700 50  0001 C CNN
+F 0 "#PWR022" H 7250 2700 50  0001 C CNN
 F 1 "GND" H 7250 2800 50  0000 C CNN
 F 2 "" H 7250 2950 50  0000 C CNN
@@
 	7250 2800 7250 2950
 $Comp
-L GND #PWR017
+L GND #PWR023
 U 1 1 59E36B34
 P 7900 2950
-F 0 "#PWR017" H 7900 2700 50  0001 C CNN
+F 0 "#PWR023" H 7900 2700 50  0001 C CNN
 F 1 "GND" H 7900 2800 50  0000 C CNN
 F 2 "" H 7900 2950 50  0000 C CNN
@@
 	2750 2150 2750 2250
 $Comp
-L GND #PWR018
+L GND #PWR024
 U 1 1 59E3722D
 P 2750 2950
-F 0 "#PWR018" H 2750 2700 50  0001 C CNN
+F 0 "#PWR024" H 2750 2700 50  0001 C CNN
 F 1 "GND" H 2750 2800 50  0000 C CNN
 F 2 "" H 2750 2950 50  0000 C CNN
@@
 Connection ~ 2050 1400
 $Comp
-L +9V #PWR019
+L +9V #PWR025
 U 1 1 59E373B1
 P 4600 1950
-F 0 "#PWR019" H 4600 1800 50  0001 C CNN
+F 0 "#PWR025" H 4600 1800 50  0001 C CNN
 F 1 "+9V" H 4600 2090 50  0000 C CNN
 F 2 "" H 4600 1950 50  0000 C CNN
@@
 	4600 2150 4000 2150
 $Comp
-L +9V #PWR020
+L +9V #PWR026
 U 1 1 59E37537
 P 2050 1200
-F 0 "#PWR020" H 2050 1050 50  0001 C CNN
+F 0 "#PWR026" H 2050 1050 50  0001 C CNN
 F 1 "+9V" H 2050 1340 50  0000 C CNN
 F 2 "" H 2050 1200 50  0000 C CNN
@@
 $EndComp
 $Comp
-L GND #PWR021
+L GND #PWR027
 U 1 1 59E378E0
 P 2050 2050
-F 0 "#PWR021" H 2050 1800 50  0001 C CNN
+F 0 "#PWR027" H 2050 1800 50  0001 C CNN
 F 1 "GND" H 2050 1900 50  0000 C CNN
 F 2 "" H 2050 2050 50  0000 C CNN
@@
 VNXE
 $Comp
-L NJM7805S U7
+L NJM7805S U9
 U 1 1 59E3AA98
 P 3650 5100
-F 0 "U7" H 3925 5225 60  0000 C CNN
+F 0 "U9" H 3925 5225 60  0000 C CNN
 F 1 "NJM7805S" H 4025 4800 60  0000 C CNN
 F 2 "TO_SOT_Packages_SMD:TO-252-3_TabPin2" H 3650 5100 60  0001 C CNN
@@
 $EndComp
 $Comp
-L C C4
+L C C5
 U 1 1 59E53D99
 P 3000 5450
-F 0 "C4" H 3025 5550 50  0000 L CNN
+F 0 "C5" H 3025 5550 50  0000 L CNN
 F 1 "0.1u" H 3025 5350 50  0000 L CNN
 F 2 "Capacitors_SMD:C_0603" H 3038 5300 50  0001 C CNN
@@
 $EndComp
 $Comp
-L C C5
+L C C6
 U 1 1 59E5422C
 P 4500 5450
-F 0 "C5" H 4525 5550 50  0000 L CNN
+F 0 "C6" H 4525 5550 50  0000 L CNN
 F 1 "0.1u" H 4525 5350 50  0000 L CNN
 F 2 "Capacitors_SMD:C_0603" H 4538 5300 50  0001 C CNN
@@
 $EndComp
 $Comp
-L CP1 C2
+L CP1 C4
 U 1 1 59E543AD
 P 2500 5450
-F 0 "C2" H 2525 5550 50  0000 L CNN
+F 0 "C4" H 2525 5550 50  0000 L CNN
 F 1 "47u" H 2525 5350 50  0000 L CNN
 F 2 "Capacitors_ThroughHole:CP_Radial_D7.5mm_P2.50mm" H 2500 5450 50  0001 C CNN
@@
 $EndComp
 $Comp
-L CP1 C6
+L CP1 C7
 U 1 1 59E546F5
 P 5050 5450
-F 0 "C6" H 5075 5550 50  0000 L CNN
+F 0 "C7" H 5075 5550 50  0000 L CNN
 F 1 "47u" H 5075 5350 50  0000 L CNN
 F 2 "Capacitors_ThroughHole:CP_Radial_D7.5mm_P2.50mm" H 5050 5450 50  0001 C CNN
@@
 $EndComp
 $Comp
-L +9V #PWR022
+L +9V #PWR028
 U 1 1 59E54EBB
 P 2500 4900
-F 0 "#PWR022" H 2500 4750 50  0001 C CNN
+F 0 "#PWR028" H 2500 4750 50  0001 C CNN
 F 1 "+9V" H 2500 5040 50  0000 C CNN
 F 2 "" H 2500 4900 50  0000 C CNN
@@
 $EndComp
 $Comp
-L +5V #PWR023
+L +5V #PWR029
 U 1 1 59E55331
 P 5050 4900
-F 0 "#PWR023" H 5050 4750 50  0001 C CNN
+F 0 "#PWR029" H 5050 4750 50  0001 C CNN
 F 1 "+5V" H 5050 5040 50  0000 C CNN
 F 2 "" H 5050 4900 50  0000 C CNN
@@
 Connection ~ 4500 5100
 $Comp
-L GND #PWR024
+L GND #PWR030
 U 1 1 59E55DA3
 P 3750 5850
-F 0 "#PWR024" H 3750 5600 50  0001 C CNN
+F 0 "#PWR030" H 3750 5600 50  0001 C CNN
 F 1 "GND" H 3750 5700 50  0000 C CNN
 F 2 "" H 3750 5850 50  0000 C CNN
@@
 Connection ~ 4500 5750
 $Comp
-L PWR_FLAG #FLG025
+L PWR_FLAG #FLG031
 U 1 1 59E57208
 P 1250 1100
-F 0 "#FLG025" H 1250 1195 50  0001 C CNN
+F 0 "#FLG031" H 1250 1195 50  0001 C CNN
 F 1 "PWR_FLAG" H 1250 1280 50  0000 C CNN
 F 2 "" H 1250 1100 50  0000 C CNN
@@
 $EndComp
 $Comp
-L +9V #PWR026
+L +9V #PWR032
 U 1 1 59E572E3
 P 850 1100
-F 0 "#PWR026" H 850 950 50  0001 C CNN
+F 0 "#PWR032" H 850 950 50  0001 C CNN
 F 1 "+9V" H 850 1240 50  0000 C CNN
 F 2 "" H 850 1100 50  0000 C CNN
@@
 	1250 1250 1250 1100
 $Comp
-L GND #PWR027
+L GND #PWR033
 U 1 1 59E58398
 P 900 1850
-F 0 "#PWR027" H 900 1600 50  0001 C CNN
+F 0 "#PWR033" H 900 1600 50  0001 C CNN
 F 1 "GND" H 900 1700 50  0000 C CNN
 F 2 "" H 900 1850 50  0000 C CNN
@@
 $EndComp
 $Comp
-L PWR_FLAG #FLG028
+L PWR_FLAG #FLG034
 U 1 1 59E58668
 P 1250 1600
-F 0 "#FLG028" H 1250 1695 50  0001 C CNN
+F 0 "#FLG034" H 1250 1695 50  0001 C CNN
 F 1 "PWR_FLAG" H 1250 1780 50  0000 C CNN
 F 2 "" H 1250 1600 50  0000 C CNN
@@
 Connection ~ 1850 4100
 $Comp
-L GND #PWR029
+L GND #PWR035
 U 1 1 59EA9E83
 P 1850 4300
-F 0 "#PWR029" H 1850 4050 50  0001 C CNN
+F 0 "#PWR035" H 1850 4050 50  0001 C CNN
 F 1 "GND" H 1850 4150 50  0000 C CNN
 F 2 "" H 1850 4300 50  0000 C CNN
@@
 $EndComp
 $Comp
-L +9V #PWR030
+L +9V #PWR036
 U 1 1 59EAA3F3
 P 1850 3600
-F 0 "#PWR030" H 1850 3450 50  0001 C CNN
+F 0 "#PWR036" H 1850 3450 50  0001 C CNN
 F 1 "+9V" H 1850 3740 50  0000 C CNN
 F 2 "" H 1850 3600 50  0000 C CNN

Commit message: add connectors
Parts:
- Q1: footprint TO_SOT_Packages_THT:TO-220-3_Vertical -> TO_SOT_Packages_THT:TO-220-3_Horizontal
Changed lines of the file:
@@
 F 0 "Q1" H 6350 2000 50  0000 R CNN
 F 1 "2SK3234" H 6600 1900 50  0000 R CNN
-F 2 "TO_SOT_Packages_THT:TO-220-3_Vertical" H 6250 2050 50  0001 C CNN
+F 2 "TO_SOT_Packages_THT:TO-220-3_Horizontal" H 6250 2050 50  0001 C CNN
 F 3 "" H 6050 1950 50  0000 C CNN
 	1    6050 1950
