File: KiCad/power.sch (KiCad schematic (older format))
At the start: 22 parts, among them CON1 BARREL_JACK, Q1 2SK3234, Q2 2SA1015, U8 NJM2360A, U9 NJM7805S

Commit message: place components
Parts:
- C4, C7: footprint Capacitors_ThroughHole:CP_Radial_D7.5mm_P2.50mm -> nixie_clock:C_3225
Changed lines of the file:
@@
 F 0 "C4" H 2525 5550 50  0000 L CNN
 F 1 "47u" H 2525 5350 50  0000 L CNN
-F 2 "Capacitors_ThroughHole:CP_Radial_D7.5mm_P2.50mm" H 2500 5450 50  0001 C CNN
+F 2 "nixie_clock:C_3225" H 2500 5450 50  0001 C CNN
 F 3 "" H 2500 5450 50  0000 C CNN
 	1    2500 5450
@@
 F 0 "C7" H 5075 5550 50  0000 L CNN
 F 1 "47u" H 5075 5350 50  0000 L CNN
-F 2 "Capacitors_ThroughHole:CP_Radial_D7.5mm_P2.50mm" H 5050 5450 50  0001 C CNN
+F 2 "nixie_clock:C_3225" H 5050 5450 50  0001 C CNN
 F 3 "" H 5050 5450 50  0000 C CNN
 	1    5050 5450

Commit message: change pcb designs
Parts:
- C2: footprint Capacitors_ThroughHole:CP_Radial_D12.5mm_P5.00mm -> Capacitors_ThroughHole:CP_Radial_D10.0mm_P5.00mm
Changed lines of the file:
@@
 $EndComp
 $Comp
-L GND #PWR018
+L GND #PWR019
 U 1 1 59E35E0E
 P 6150 2950
-F 0 "#PWR018" H 6150 2700 50  0001 C CNN
+F 0 "#PWR019" H 6150 2700 50  0001 C CNN
 F 1 "GND" H 6150 2800 50  0000 C CNN
 F 2 "" H 6150 2950 50  0000 C CNN
@@
 $EndComp
 $Comp
-L GND #PWR019
+L GND #PWR020
 U 1 1 59E35F44
 P 5000 2950
-F 0 "#PWR019" H 5000 2700 50  0001 C CNN
+F 0 "#PWR020" H 5000 2700 50  0001 C CNN
 F 1 "GND" H 5000 2800 50  0000 C CNN
 F 2 "" H 5000 2950 50  0000 C CNN
@@
 F 0 "C2" H 7925 1850 50  0000 L CNN
 F 1 "10u/400V" H 7925 1650 50  0000 L CNN
-F 2 "Capacitors_ThroughHole:CP_Radial_D12.5mm_P5.00mm" H 7900 1750 50  0001 C CNN
+F 2 "Capacitors_ThroughHole:CP_Radial_D10.0mm_P5.00mm" H 7900 1750 50  0001 C CNN
 F 3 "" H 7900 1750 50  0000 C CNN
 	1    7900 1750
@@
 $EndComp
 $Comp
-L GND #PWR020
+L GND #PWR021
 U 1 1 59E3695E
 P 7250 2950
-F 0 "#PWR020" H 7250 2700 50  0001 C CNN
+F 0 "#PWR021" H 7250 2700 50  0001 C CNN
 F 1 "GND" H 7250 2800 50  0000 C CNN
 F 2 "" H 7250 2950 50  0000 C CNN
@@
 	7250 2800 7250 2950
 $Comp
-L GND #PWR021
+L GND #PWR022
 U 1 1 59E36B34
 P 7900 2950
-F 0 "#PWR021" H 7900 2700 50  0001 C CNN
+F 0 "#PWR022" H 7900 2700 50  0001 C CNN
 F 1 "GND" H 7900 2800 50  0000 C CNN
 F 2 "" H 7900 2950 50  0000 C CNN
@@
 	2750 2150 2750 2250
 $Comp
-L GND #PWR022
+L GND #PWR023
 U 1 1 59E3722D
 P 2750 2950
-F 0 "#PWR022" H 2750 2700 50  0001 C CNN
+F 0 "#PWR023" H 2750 2700 50  0001 C CNN
 F 1 "GND" H 2750 2800 50  0000 C CNN
 F 2 "" H 2750 2950 50  0000 C CNN
@@
 Connection ~ 2050 1400
 $Comp
-L +9V #PWR023
+L +9V #PWR024
 U 1 1 59E373B1
 P 4600 1950
-F 0 "#PWR023" H 4600 1800 50  0001 C CNN
+F 0 "#PWR024" H 4600 1800 50  0001 C CNN
 F 1 "+9V" H 4600 2090 50  0000 C CNN
 F 2 "" H 4600 1950 50  0000 C CNN
@@
 	4600 2150 4000 2150
 $Comp
-L +9V #PWR024
+L +9V #PWR025
 U 1 1 59E37537
 P 2050 1200
-F 0 "#PWR024" H 2050 1050 50  0001 C CNN
+F 0 "#PWR025" H 2050 1050 50  0001 C CNN
 F 1 "+9V" H 2050 1340 50  0000 C CNN
 F 2 "" H 2050 1200 50  0000 C CNN
@@
 $EndComp
 $Comp
-L GND #PWR025
+L GND #PWR026
 U 1 1 59E378E0
 P 2050 2050
-F 0 "#PWR025" H 2050 1800 50  0001 C CNN
+F 0 "#PWR026" H 2050 1800 50  0001 C CNN
 F 1 "GND" H 2050 1900 50  0000 C CNN
 F 2 "" H 2050 2050 50  0000 C CNN
@@
 $EndComp
 $Comp
-L +9V #PWR026
+L +9V #PWR027
 U 1 1 59E54EBB
 P 2500 4900
-F 0 "#PWR026" H 2500 4750 50  0001 C CNN
+F 0 "#PWR027" H 2500 4750 50  0001 C CNN
 F 1 "+9V" H 2500 5040 50  0000 C CNN
 F 2 "" H 2500 4900 50  0000 C CNN
@@
 $EndComp
 $Comp
-L +5V #PWR027
+L +5V #PWR028
 U 1 1 59E55331
 P 5050 4900
-F 0 "#PWR027" H 5050 4750 50  0001 C CNN
+F 0 "#PWR028" H 5050 4750 50  0001 C CNN
 F 1 "+5V" H 5050 5040 50  0000 C CNN
 F 2 "" H 5050 4900 50  0000 C CNN
@@
 Connection ~ 4500 5100
 $Comp
-L GND #PWR028
+L GND #PWR029
 U 1 1 59E55DA3
 P 3750 5850
-F 0 "#PWR028" H 3750 5600 50  0001 C CNN
+F 0 "#PWR029" H 3750 5600 50  0001 C CNN
 F 1 "GND" H 3750 5700 50  0000 C CNN
 F 2 "" H 3750 5850 50  0000 C CNN
@@
 Connection ~ 4500 5750
 $Comp
-L PWR_FLAG #FLG029
+L PWR_FLAG #FLG030
 U 1 1 59E57208
 P 1250 1100
-F 0 "#FLG029" H 1250 1195 50  0001 C CNN
+F 0 "#FLG030" H 1250 1195 50  0001 C CNN
 F 1 "PWR_FLAG" H 1250 1280 50  0000 C CNN
 F 2 "" H 1250 1100 50  0000 C CNN
@@
 $EndComp
 $Comp
-L +9V #PWR030
+L +9V #PWR031
 U 1 1 59E572E3
 P 850 1100
-F 0 "#PWR030" H 850 950 50  0001 C CNN
+F 0 "#PWR031" H 850 950 50  0001 C CNN
 F 1 "+9V" H 850 1240 50  0000 C CNN
 F 2 "" H 850 1100 50  0000 C CNN
@@
 	1250 1250 1250 1100
 $Comp
-L GND #PWR031
+L GND #PWR032
 U 1 1 59E58398
 P 900 1850
-F 0 "#PWR031" H 900 1600 50  0001 C CNN
+F 0 "#PWR032" H 900 1600 50  0001 C CNN
 F 1 "GND" H 900 1700 50  0000 C CNN
 F 2 "" H 900 1850 50  0000 C CNN
@@
 $EndComp
 $Comp
-L PWR_FLAG #FLG032
+L PWR_FLAG #FLG033
 U 1 1 59E58668
 P 1250 1600
-F 0 "#FLG032" H 1250 1695 50  0001 C CNN
+F 0 "#FLG033" H 1250 1695 50  0001 C CNN
 F 1 "PWR_FLAG" H 1250 1780 50  0000 C CNN
 F 2 "" H 1250 1600 50  0000 C CNN
@@
 Connection ~ 1850 4100
 $Comp
-L GND #PWR033
+L GND #PWR034
 U 1 1 59EA9E83
 P 1850 4300
-F 0 "#PWR033" H 1850 4050 50  0001 C CNN
+F 0 "#PWR034" H 1850 4050 50  0001 C CNN
 F 1 "GND" H 1850 4150 50  0000 C CNN
 F 2 "" H 1850 4300 50  0000 C CNN
@@
 $EndComp
 $Comp
-L +9V #PWR034
+L +9V #PWR035
 U 1 1 59EAA3F3
 P 1850 3600
-F 0 "#PWR034" H 1850 3450 50  0001 C CNN
+F 0 "#PWR035" H 1850 3450 50  0001 C CNN
 F 1 "+9V" H 1850 3740 50  0000 C CNN
 F 2 "" H 1850 3600 50  0000 C CNN
