File: KiCad/nixie_clock.kicad_pcb (KiCad board)
At the start: 4 copper layers, 186 x 100 mm, 72 parts, among them CON1 BARREL_JACK, P1 CONN_02X05, P2 CONN_02X05, P3 CONN_02X05, P4 CONN_02X05, Q1 2SK3234, Q2 2SA1015, U1 ESP32-DevKitC, U2 TLP627-2, U3 TLP627-2, U4 TLP627-2, U5 SN74141, U6 TLP627, U7 TLP627-2, U8 NJM2360A, U9 NJM7805S

Commit message: change pcb designs
Parts:
- C1: moved to B.Cu
- C2: footprint Capacitors_ThroughHole:CP_Radial_D12.5mm_P5.00mm -> Capacitors_ThroughHole:CP_Radial_D10.0mm_P5.00mm; moved to B.Cu
- moved R19 268.9 mm to (76.2, 145.8)
- moved R20 268.9 mm to (44.7, 148.3)
- moved R21 268.9 mm to (41.7, 143.5)
- moved R22 268.9 mm to (40.9, 148.6)
- moved R23 268.9 mm to (41.7, 136.4)
- moved R6 210.4 mm to (127.5, 131.1)
- moved R1 210.4 mm to (128.8, 178.3)
- moved R11 210.4 mm to (108.5, 137.4)
- moved R2 210.4 mm to (128.8, 170.9)
- moved R3 210.4 mm to (128.3, 157.7)
- moved R4 210.4 mm to (128.3, 150.4)
- moved R10 210.4 mm to (104.4, 151.9)
- moved R12 210.4 mm to (107.4, 131.8)
- moved R5 210.4 mm to (127.0, 137.4)
- moved R7 210.4 mm to (105.9, 178.1)
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Connections:
- P1 pad 10: /nixie/n6 -> /nixie/n3
- P1 pad 3: /nixie/n2 -> /nixie/n5
- P1 pad 4: /nixie/n9 -> /nixie/n8
- P1 pad 5: /nixie/n3 -> /nixie/n4
- P1 pad 6: /nixie/n8 -> /nixie/n9
- P1 pad 7: /nixie/n4 -> /nixie/n6
- P1 pad 8: /nixie/n7 -> /nixie/n2
- P1 pad 9: /nixie/n5 -> /nixie/n7
- P2 pad 10: /nixie/nm6 -> /nixie/nm3
- P2 pad 3: /nixie/nm2 -> /nixie/nm5
- P2 pad 4: /nixie/nm9 -> /nixie/nm8
- P2 pad 5: /nixie/nm3 -> /nixie/nm4
- P2 pad 6: /nixie/nm8 -> /nixie/nm9
- P2 pad 7: /nixie/nm4 -> /nixie/nm6
- P2 pad 8: /nixie/nm7 -> /nixie/nm2
- P2 pad 9: /nixie/nm5 -> /nixie/nm7
- P4 pad 10: /nixie/nmgnd -> GND
Routing:
- net GND: track 26.7 -> 176.4 mm, vias 0 -> 1
- net /nixie/nmc2: track 0.00 -> 69.6 mm
- net /nixie/nmc3: track 0.00 -> 68.4 mm
- net /nixie/nmc1: track 0.00 -> 67.6 mm
- net +9V: track 6.35 -> 67.7 mm
- net /nixie/nmc4: track 0.00 -> 60.7 mm
- net /nixie/nmc0: track 0.00 -> 60.0 mm
- net Net-(L1-Pad1): track 0.00 -> 55.9 mm, vias 0 -> 1
- net /nixie/nmc5: track 0.00 -> 52.9 mm
- net VNXE: track 0.00 -> 50.2 mm
- net /nixie/nmcol1: track 0.00 -> 49.9 mm
- net /nixie/nmcol0: track 0.00 -> 49.4 mm
- net /nixie/nmdot: track 0.00 -> 49.1 mm
- net /nixie/nm9: track 0.00 -> 46.6 mm
- net Net-(D7-Pad2): track 0.00 -> 42.3 mm
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