File: KiCad/nixie_clock.kicad_pcb (KiCad board)
At the start: 4 copper layers, 186 x 100 mm, 72 parts, among them CON1 BARREL_JACK, P1 CONN_02X05, P2 CONN_02X05, P3 CONN_02X05, P4 CONN_02X05, Q1 2SK3234, Q2 2SA1015, U1 ESP32-DevKitC, U2 TLP627-2, U3 TLP627-2, U4 TLP627-2, U5 SN74141, U6 TLP627, U7 TLP627-2, U8 NJM2360A, U9 NJM7805S

Commit message: finish route
Parts:
- moved R21 120.5 mm to (152.1, 95.5)
- moved R23 119.9 mm to (152.1, 89.9)
- moved R22 116.2 mm to (142.2, 91.7)
- moved R20 111.8 mm to (142.2, 93.7)
- moved R1 78.1 mm to (176.0, 116.1), turned to 180 degrees
- moved U6 76.6 mm to (155.4, 119.9), turned to 90 degrees
- moved R19 73.3 mm to (142.2, 114.0)
- moved R7 70.1 mm to (142.2, 118.1)
- moved R2 69.0 mm to (176.0, 120.7), turned to 180 degrees
- moved R11 68.1 mm to (142.2, 78.2)
- moved R9 64.8 mm to (142.2, 104.9)
- moved R8 64.5 mm to (142.2, 120.1)
- moved R5 64.3 mm to (152.1, 78.2)
- moved U3 63.8 mm to (160.5, 109.2)
- moved R12 62.2 mm to (142.2, 80.3)
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Connections:
- U1 pad 24: nxeb -> nxed
- U1 pad 25: nxec -> nxeb
- U1 pad 26: nxed -> nxec
- U2 pad 1: Net-(R7-Pad2) -> Net-(R8-Pad2)
- U2 pad 2: nxecom0 -> nxecom1
- U2 pad 3: Net-(R8-Pad2) -> Net-(R7-Pad2)
- U2 pad 4: nxecom1 -> nxecom0
- U2 pad 5: /nixie/nmc1 -> /nixie/nmc0
- U2 pad 6: Net-(R2-Pad2) -> Net-(R1-Pad2)
- U2 pad 7: /nixie/nmc0 -> /nixie/nmc1
- U2 pad 8: Net-(R1-Pad2) -> Net-(R2-Pad2)
- U4 pad 1: Net-(R11-Pad2) -> Net-(R12-Pad2)
- U4 pad 2: nxecom4 -> nxecom5
- U4 pad 3: Net-(R12-Pad2) -> Net-(R11-Pad2)
- U4 pad 4: nxecom5 -> nxecom4
- U4 pad 5: /nixie/nmc5 -> /nixie/nmc4
- U4 pad 6: Net-(R6-Pad2) -> Net-(R5-Pad2)
- U4 pad 7: /nixie/nmc4 -> /nixie/nmc5
- U4 pad 8: Net-(R5-Pad2) -> Net-(R6-Pad2)
Routing:
- net +3V3: track 0.00 -> 297.8 mm, vias 0 -> 1
- net GND: track 176.4 -> 362.7 mm, vias 1 -> 12
- net +5V: track 6.60 -> 192.6 mm
- net VNXE: track 50.2 -> 191.8 mm
- net led5: track 0.00 -> 123.5 mm
- net nxecom1: track 0.00 -> 93.9 mm, vias 0 -> 1
- net led4: track 0.00 -> 88.9 mm, vias 0 -> 1
- net nxecom0: track 0.00 -> 84.0 mm
- net nxecom2: track 0.00 -> 70.4 mm
- net nxecom3: track 0.00 -> 69.7 mm
- net nxea: track 0.00 -> 60.5 mm
- net led3: track 0.00 -> 60.0 mm, vias 0 -> 1
- net nxedot: track 0.00 -> 59.4 mm, vias 0 -> 1
- net nxecom4: track 0.00 -> 59.0 mm
- net nxed: track 0.00 -> 56.9 mm
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- added copper zone on In2.Cu, net +3V3
- added copper zone on B.Cu, net /nixie/ngnd
- added copper zone on F.Cu, net /nixie/ngnd
- added copper zone on F.Cu, net GND
- added copper zone on In1.Cu, net GND

Commit message: change pcb
Parts:
- moved C1 2.24 mm to (230.1, 89.1)
- moved C2 2.24 mm to (183.6, 95.0)
- moved C3 2.24 mm to (206.2, 83.5)
- moved C4 2.24 mm to (217.7, 120.6)
- moved C5 2.24 mm to (212.1, 124.7)
- moved C6 2.24 mm to (209.0, 124.7)
- moved C7 2.24 mm to (203.7, 120.6)
- moved CON1 2.24 mm to (226.8, 115.0)
- moved D1 2.24 mm to (81.0, 102.0)
- moved D2 2.24 mm to (103.0, 102.0)
- moved D3 2.24 mm to (133.0, 102.0)
- moved D4 2.24 mm to (155.0, 102.0)
- moved D5 2.24 mm to (185.0, 102.0)
- moved D6 2.24 mm to (207.0, 102.0)
- moved D7 2.24 mm to (178.8, 110.5)
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Routing:
- net /nixie/ngnd: track 120.1 -> 547.6 mm, vias 0 -> 16
- added copper zone on B.Cu, net GND
