File: KiCad/ESP32.sch (KiCad schematic (older format))
At the start: 1 part

Commit message: add power schematic
Parts:
- removed U?: ESP32-WROOM, ESP32-footprints-Lib:ESP32-WROOM, symbol ESP32-WROOM
- added U?: ESP32-DevKitC, symbol ESP32-DevKitC
Connections:
- net labels added: +3.3V, +5V, GND
- wire segments 0 -> 9
Changed lines of the file:
@@
 encoding utf-8
 Sheet 2 4
-Title ""
-Date ""
+Title "ESP32"
+Date "2017-10-16"
 Rev ""
 Comp ""
@@
 $EndDescr
 $Comp
-L ESP32-WROOM U?
-U 1 1 59E23973
-P 4700 2950
-F 0 "U?" H 4000 4200 60  0000 C CNN
-F 1 "ESP32-WROOM" H 5200 4200 60  0000 C CNN
-F 2 "ESP32-footprints-Lib:ESP32-WROOM" H 5050 4300 60  0001 C CNN
-F 3 "" H 4250 3400 60  0001 C CNN
-	1    4700 2950
+L ESP32-DevKitC U?
+U 1 1 59E597A2
+P 2750 1650
+F 0 "U?" H 3150 -350 60  0000 C CNN
+F 1 "ESP32-DevKitC" H 3150 1750 60  0000 C CNN
+F 2 "" H 3200 1350 60  0000 C CNN
+F 3 "" H 3200 1350 60  0000 C CNN
+	1    2750 1650
 	1    0    0    -1
 $EndComp
+$Comp
+L +5V #PWR?
+U 1 1 59E598C7
+P 1750 3400
+F 0 "#PWR?" H 1750 3250 50  0001 C CNN
+F 1 "+5V" H 1750 3540 50  0000 C CNN
+F 2 "" H 1750 3400 50  0000 C CNN
+F 3 "" H 1750 3400 50  0000 C CNN
+	1    1750 3400
+	1    0    0    -1
+$EndComp
+Wire Wire Line
+	2550 3500 1750 3500
+Wire Wire Line
+	1750 3500 1750 3400
+$Comp
+L GND #PWR?
+U 1 1 59E598FC
+P 4800 2500
+F 0 "#PWR?" H 4800 2250 50  0001 C CNN
+F 1 "GND" H 4800 2350 50  0000 C CNN
+F 2 "" H 4800 2500 50  0000 C CNN
+F 3 "" H 4800 2500 50  0000 C CNN
+	1    4800 2500
+	1    0    0    -1
+$EndComp
+Wire Wire Line
+	3750 2300 4800 2300
+Wire Wire Line
+	4800 1700 4800 2500
+Wire Wire Line
+	3750 1700 4800 1700
+Connection ~ 4800 2300
+$Comp
+L +3.3V #PWR?
+U 1 1 59E5991F
+P 1750 1550
+F 0 "#PWR?" H 1750 1400 50  0001 C CNN
+F 1 "+3.3V" H 1750 1690 50  0000 C CNN
+F 2 "" H 1750 1550 50  0000 C CNN
+F 3 "" H 1750 1550 50  0000 C CNN
+	1    1750 1550
+	1    0    0    -1
+$EndComp
+Wire Wire Line
+	1750 1550 1750 1700
+Wire Wire Line
+	1750 1700 2550 1700
+$Comp
+L GND #PWR?
+U 1 1 59E5993D
+P 2050 3050
+F 0 "#PWR?" H 2050 2800 50  0001 C CNN
+F 1 "GND" H 2050 2900 50  0000 C CNN
+F 2 "" H 2050 3050 50  0000 C CNN
+F 3 "" H 2050 3050 50  0000 C CNN
+	1    2050 3050
+	1    0    0    -1
+$EndComp
+Wire Wire Line
+	2050 3050 2050 3000
+Wire Wire Line
+	2050 3000 2550 3000
 $EndSCHEMATC

Commit message: change schematics
Parts:
- gave numbers to parts that had none: 1
Connections:
- net nxecom5: now reaches U1.10 (IO26)
- net nxea: now reaches U1.23 (IO15)
- net nxeb: now reaches U1.24 (IO2)
- net nxec: now reaches U1.25 (IO0)
- net nxed: now reaches U1.26 (IO4)
- net nxecom0: now reaches U1.5 (IO34)
- net nxecom1: now reaches U1.6 (IO35)
- net nxecom2: now reaches U1.7 (IO32)
- net nxecom3: now reaches U1.8 (IO33)
- net nxecom4: now reaches U1.9 (IO25)
- no-connect marks 0 -> 23
Changed lines of the file:
@@
 $EndDescr
 $Comp
-L ESP32-DevKitC U?
+L ESP32-DevKitC U1
 U 1 1 59E597A2
 P 2750 1650
-F 0 "U?" H 3150 -350 60  0000 C CNN
+F 0 "U1" H 3150 -350 60  0000 C CNN
 F 1 "ESP32-DevKitC" H 3150 1750 60  0000 C CNN
 F 2 "" H 3200 1350 60  0000 C CNN
@@
 $EndComp
 $Comp
-L +5V #PWR?
+L +5V #PWR01
 U 1 1 59E598C7
 P 1750 3400
-F 0 "#PWR?" H 1750 3250 50  0001 C CNN
+F 0 "#PWR01" H 1750 3250 50  0001 C CNN
 F 1 "+5V" H 1750 3540 50  0000 C CNN
 F 2 "" H 1750 3400 50  0000 C CNN
@@
 	1750 3500 1750 3400
 $Comp
-L GND #PWR?
+L GND #PWR02
 U 1 1 59E598FC
 P 4800 2500
-F 0 "#PWR?" H 4800 2250 50  0001 C CNN
+F 0 "#PWR02" H 4800 2250 50  0001 C CNN
 F 1 "GND" H 4800 2350 50  0000 C CNN
 F 2 "" H 4800 2500 50  0000 C CNN
@@
 Connection ~ 4800 2300
 $Comp
-L +3.3V #PWR?
+L +3.3V #PWR03
 U 1 1 59E5991F
 P 1750 1550
-F 0 "#PWR?" H 1750 1400 50  0001 C CNN
+F 0 "#PWR03" H 1750 1400 50  0001 C CNN
 F 1 "+3.3V" H 1750 1690 50  0000 C CNN
 F 2 "" H 1750 1550 50  0000 C CNN
@@
 	1750 1700 2550 1700
 $Comp
-L GND #PWR?
+L GND #PWR04
 U 1 1 59E5993D
 P 2050 3050
-F 0 "#PWR?" H 2050 2800 50  0001 C CNN
+F 0 "#PWR04" H 2050 2800 50  0001 C CNN
 F 1 "GND" H 2050 2900 50  0000 C CNN
 F 2 "" H 2050 3050 50  0000 C CNN
@@
 Wire Wire Line
 	2050 3000 2550 3000
+Text GLabel 2250 2100 0    60   Output ~ 0
+nxecom0
+Text GLabel 2250 2200 0    60   Output ~ 0
+nxecom1
+Text GLabel 2250 2300 0    60   Output ~ 0
+nxecom2
+Text GLabel 2250 2400 0    60   Output ~ 0
+nxecom3
+Text GLabel 2250 2500 0    60   Output ~ 0
+nxecom4
+Text GLabel 2250 2600 0    60   Output ~ 0
+nxecom5
+Text GLabel 4000 3200 2    60   Output ~ 0
+nxea
+Text GLabel 4000 3100 2    60   Output ~ 0
+nxeb
+Text GLabel 4000 3000 2    60   Output ~ 0
+nxec
+Text GLabel 4000 2900 2    60   Output ~ 0
+nxed
+Wire Wire Line
+	2250 2100 2550 2100
+Wire Wire Line
+	2250 2200 2550 2200
+Wire Wire Line
+	2250 2300 2550 2300
+Wire Wire Line
+	2250 2400 2550 2400
+Wire Wire Line
+	2250 2500 2550 2500
+Wire Wire Line
+	2250 2600 2550 2600
+Wire Wire Line
+	3750 3200 4000 3200
+Wire Wire Line
+	3750 3100 4000 3100
+Wire Wire Line
+	3750 3000 4000 3000
+Wire Wire Line
+	3750 2900 4000 2900
+NoConn ~ 2550 1800
+NoConn ~ 2550 1900
+NoConn ~ 2550 2000
+NoConn ~ 2550 2700
+NoConn ~ 2550 2800
+NoConn ~ 2550 2900
+NoConn ~ 2550 3100
+NoConn ~ 2550 3200
+NoConn ~ 2550 3300
+NoConn ~ 2550 3400
+NoConn ~ 3750 3500
+NoConn ~ 3750 3400
+NoConn ~ 3750 3300
+NoConn ~ 3750 2800
+NoConn ~ 3750 2700
+NoConn ~ 3750 2600
+NoConn ~ 3750 2500
+NoConn ~ 3750 2400
+NoConn ~ 3750 2200
+NoConn ~ 3750 2100
+NoConn ~ 3750 2000
+NoConn ~ 3750 1900
+NoConn ~ 3750 1800
 $EndSCHEMATC

Commit message: add pcb design
Parts:
- U1: footprint (none) -> nixie_clock:ESP32-DEV-Kit
Changed lines of the file:
@@
 F 0 "U1" H 3150 -350 60  0000 C CNN
 F 1 "ESP32-DevKitC" H 3150 1750 60  0000 C CNN
-F 2 "" H 3200 1350 60  0000 C CNN
+F 2 "nixie_clock:ESP32-DEV-Kit" H 3200 1350 60  0001 C CNN
 F 3 "" H 3200 1350 60  0000 C CNN
 	1    2750 1650

Commit message: change schematics
Connections:
- net led5: now reaches U1.29 (IO5)
- net led4: now reaches U1.30 (IO18)
- net led3: now reaches U1.31 (IO19)
- net led2: now reaches U1.33 (IO21)
- net led1: now reaches U1.36 (IO22)
- net led0: now reaches U1.37 (IO23)
- no-connect marks 23 -> 17
Changed lines of the file:
@@
 NoConn ~ 3750 2800
 NoConn ~ 3750 2700
-NoConn ~ 3750 2600
-NoConn ~ 3750 2500
-NoConn ~ 3750 2400
-NoConn ~ 3750 2200
 NoConn ~ 3750 2100
 NoConn ~ 3750 2000
-NoConn ~ 3750 1900
-NoConn ~ 3750 1800
+Text GLabel 4000 1800 2    60   Output ~ 0
+led0
+Text GLabel 4000 1900 2    60   Output ~ 0
+led1
+Text GLabel 4000 2200 2    60   Output ~ 0
+led2
+Text GLabel 4000 2400 2    60   Output ~ 0
+led3
+Text GLabel 4000 2500 2    60   Output ~ 0
+led4
+Text GLabel 4000 2600 2    60   Output ~ 0
+led5
+Wire Wire Line
+	3750 1800 4000 1800
+Wire Wire Line
+	3750 1900 4000 1900
+Wire Wire Line
+	3750 2200 4000 2200
+Wire Wire Line
+	3750 2600 4000 2600
+Wire Wire Line
+	3750 2500 4000 2500
+Wire Wire Line
+	3750 2400 4000 2400
 $EndSCHEMATC

Commit message: many changes
Connections:
- net nxedot: now reaches U1.11 (IO27)
- net nxecol0: now reaches U1.12 (IO14)
- net nxecol1: now reaches U1.13 (IO12)
- no-connect marks 17 -> 14
Changed lines of the file:
@@
 NoConn ~ 2550 1900
 NoConn ~ 2550 2000
-NoConn ~ 2550 2700
-NoConn ~ 2550 2800
-NoConn ~ 2550 2900
 NoConn ~ 2550 3100
 NoConn ~ 2550 3200
@@
 Wire Wire Line
 	3750 2400 4000 2400
+Text GLabel 2250 2700 0    60   Output ~ 0
+nxedot
+Text GLabel 2250 2800 0    60   Output ~ 0
+nxecol0
+Text GLabel 2250 2900 0    60   Output ~ 0
+nxecol1
+Wire Wire Line
+	2250 2700 2550 2700
+Wire Wire Line
+	2250 2800 2550 2800
+Wire Wire Line
+	2250 2900 2550 2900
 $EndSCHEMATC

Commit message: finish route
Connections:
- net nxeb: now also U1.25 (IO0); no longer U1.24 (IO2)
- net nxec: now also U1.26 (IO4); no longer U1.25 (IO0)
- net nxed: now also U1.24 (IO2); no longer U1.26 (IO4)
Changed lines of the file:
@@
 Text GLabel 4000 3200 2    60   Output ~ 0
 nxea
+Text GLabel 4000 3000 2    60   Output ~ 0
+nxeb
+Text GLabel 4000 2900 2    60   Output ~ 0
+nxec
 Text GLabel 4000 3100 2    60   Output ~ 0
-nxeb
-Text GLabel 4000 3000 2    60   Output ~ 0
-nxec
-Text GLabel 4000 2900 2    60   Output ~ 0
 nxed
 Wire Wire Line
